File: DAC.sch (KiCad schematic (older format))
At the start: 16 parts, among them Q1 MJD31CT4G, U3 MCP4728, U4 TLV2371

Commit message: Changed 47R resistor part number
Parts:
- R7: Manufacturer Walsin -> Multicomp; Order Code 2502729 -> 2447666; Part Number WR08X47R0FTL -> MCWR08X47R0FTL
Changed lines of the file:
@@
 F 2 "Resistors_SMD:R_0805" V 9280 2400 50  0001 C CNN
 F 3 "" H 9350 2400 50  0000 C CNN
-F 4 "WR08X47R0FTL" H 9350 2400 60  0001 C CNN "Part Number"
-F 5 "Walsin" H 9350 2400 60  0001 C CNN "Manufacturer"
+F 4 "MCWR08X47R0FTL" H 9350 2400 60  0001 C CNN "Part Number"
+F 5 "Multicomp" H 9350 2400 60  0001 C CNN "Manufacturer"
 F 6 "0805" H 9350 2400 60  0001 C CNN "Package"
 F 7 "Farnell" H 9350 2400 60  0001 C CNN "Supplier"
-F 8 "2502729" H 9350 2400 60  0001 C CNN "Order Code"
+F 8 "2447666" H 9350 2400 60  0001 C CNN "Order Code"
 F 9 "Mouser" H 9350 2400 60  0001 C CNN "Alt. Supplier"
 F 10 "667-ERJ-6GEYJ470V" H 9350 2400 60  0001 C CNN "Alt. Order Code"
